Commit message: adding noise to simulation

File: rotors_simulator/rotors_description/urdf/R_bebop2.xacro (robot description, xacro)
@@ -16,23 +16,15 @@
   limitations under the License.
 -->
-<robot name="$(arg mav_name)" xmlns:xacro="http://ros.org/wiki/xacro">
+<robot name="bebop2" xmlns:xacro="http://ros.org/wiki/xacro">
   <!-- Instantiate the mav-->
-  <xacro:include filename="$(find rotors_description)/urdf/$(arg mav_name)_base_modified.xacro" />
-  <link name="world"/>
-  <joint name="world_right_base_joint" type="fixed">
-    <parent link="world"/>
-    <child link="R_${namespace}/base_link"/>
-    <origin xyz="0.0 0.5 0.05" rpy="0.0 0.0 0.0"/>
-  </joint>
-  <joint name="world_left_base_joint" type="fixed">
-    <parent link="world"/>
-    <child link="L_${namespace}/base_link"/>
-    <origin xyz="0.0 -0.5 0.05" rpy="0.0 0.0 0.0"/>
-  </joint>
+  <xacro:property name="namespace" value="bebop2" />
+  <xacro:include filename="$(find rotors_description)/urdf/bebop2_base.xacro">
+  <xacro:arg name="namespace" value="bebop2" />
+  </xacro:include>
   <!-- Mount a generic odometry sensor without odometry map (working everywhere). -->
   <xacro:odometry_plugin_macro
-    namespace="R_${namespace}"
+    namespace="${namespace}"
     odometry_sensor_suffix="1"
-    parent_link="R_${namespace}/base_link"
+    parent_link="${namespace}/base_link"
     pose_topic="odometry_sensor1/pose"
     pose_with_covariance_topic="odometry_sensor1/pose_with_covariance"
@@ -41,35 +33,5 @@
     odometry_topic="odometry_sensor1/odometry"
     parent_frame_id="world"
-    child_frame_id="R_${namespace}/odometry_sensor1"
-    mass_odometry_sensor="0.00001"
-    measurement_divisor="1"
-    measurement_delay="0"
-    unknown_delay="0.0"
-    noise_normal_position="0 0 0"
-    noise_normal_quaternion="0 0 0"
-    noise_normal_linear_velocity="0 0 0"
-    noise_normal_angular_velocity="0 0 0"
-    noise_uniform_position="0 0 0"
-    noise_uniform_quaternion="0 0 0"
-    noise_uniform_linear_velocity="0 0 0"
-    noise_uniform_angular_velocity="0 0 0"
-    enable_odometry_map="false"
-    odometry_map=""
-    image_scale="">
-    <inertia ixx="0.00001" ixy="0.0" ixz="0.0" iyy="0.00001" iyz="0.0" izz="0.00001" /> <!-- [kg m^2] [kg m^2] [kg m^2] [kg m^2] [kg m^2] [kg m^2] -->
-    <origin xyz="0.0 0.0 0.0" rpy="0.0 0.0 0.0" />
-  </xacro:odometry_plugin_macro>
-    <!-- Mount a generic odometry sensor without odometry map (working everywhere). -->
-    <xacro:odometry_plugin_macro
-    namespace="L_${namespace}"
-    odometry_sensor_suffix="1"
-    parent_link="L_${namespace}/base_link"
-    pose_topic="odometry_sensor1/pose"
-    pose_with_covariance_topic="odometry_sensor1/pose_with_covariance"
-    position_topic="odometry_sensor1/position"
-    transform_topic="odometry_sensor1/transform"
-    odometry_topic="odometry_sensor1/odometry"
-    parent_frame_id="world"
-    child_frame_id="L_${namespace}/odometry_sensor1"
+    child_frame_id="${namespace}/odometry_sensor1"
     mass_odometry_sensor="0.00001"
     measurement_divisor="1"
